Commit message: push to github

File: src/gazebo/launch/env.urdf (robot description, URDF)
Before this commit: robot environment, 12 links, 11 joints
Links:
- removed link box1_link
- removed link box2_link
- removed link box3_link
- removed link box4_link
- removed link box5_link
- removed link cyl1_link
- removed link cyl2_link
- removed link sim_world
- removed link wall1_link
- removed link wall2_link
- removed link wall3_link
- removed link wall4_link
- added link box1; visual box size=3 3 3.0
- added link box2; visual box size=3 3 3.0
- added link box3; visual box size=3 3 3.0
- added link box4; visual box size=2 2 3.0
- added link box5; visual box size=2 2 3.0
- added link cyl1; visual cylinder length=3 radius=3
- added link cyl2; visual cylinder length=3 radius=2
- added link wall; visual box size=30 0.5 3.0
- added link wall1; visual box size=30 0.5 3.0
- added link wall2; visual box size=0.5 30 3.0
- added link wall3; visual box size=0.5 30 3.0
Joints:
- removed joint box1_joint
- removed joint box2_joint
- removed joint box3_joint
- removed joint box4_joint
- removed joint box5_joint
- removed joint cyl1_joint
- removed joint cyl2_joint
- removed joint wall1_joint
- removed joint wall2_joint
- removed joint wall3_joint
- removed joint wall4_joint
- added joint j1: type fixed, parent sim_world, child wall, origin xyz=0 -15 0
- added joint j10: type fixed, parent sim_world, child cyl1, origin xyz=0 0 0
- added joint j11: type fixed, parent sim_world, child cyl2, origin xyz=-7 -7 0
- added joint j2: type fixed, parent sim_world, child wall1, origin xyz=0 15 0
- added joint j3: type fixed, parent sim_world, child wall2, origin xyz=15 0 0
- added joint j4: type fixed, parent sim_world, child wall3, origin xyz=-15 0 0
- added joint j5: type fixed, parent sim_world, child box1, origin xyz=7 -6 0
- added joint j6: type fixed, parent sim_world, child box2, origin xyz=-8 6 0
- added joint j7: type fixed, parent sim_world, child box3, origin xyz=4 9 0
- added joint j8: type fixed, parent sim_world, child box4, origin xyz=9 3 0
- added joint j9: type fixed, parent sim_world, child box5, origin xyz=1 -10 0
